File: eagle/base.brd (EAGLE design)
At the start: 105.1 x 83.8 mm, 71 parts, among them IC1 FM22L16-55-TG, IC2 ATSAMS70Q21A-AN, IC3 MFS401N-2-Z, IC4 ADT7310TRZ

Commit message: Update to version 2
Parts:
- removed C1, C5: 4.7uF, rcl:C0603
- removed C18, C19: (no value), rcl:C0603
- removed IC3: MFS401N-2-Z, MFS401N-2-Z:MFS401N2Z
- removed JPCORE, JPMAIN, JPVDD: (no value), pinhead:1X02
- removed LED9: (no value), led:CHIP-LED0603
- removed Q1: (no value), crystal:HC49/S
- added C21: 100nF, rcl:C0603
- added C22, C24: 470pF, rcl:C0603
- added C23, C25: 2.2uF, rcl:C0603
- added C26, C27: 1uF, rcl:C0603
- added DBG_ON, LED_2.2, LED_VAR: KPHD-1608LVCGCK, led:CHIP-LED0603
- added FL1, FL2: MIC5205YM5-TR, MIC5205YM5-TR:SOT95P280X145-5N
- added JP1, USBALIM: (no value), pinhead:1X02
- added R17: 100k, rcl:R0603
- added R18: 76.8k, rcl:R0603
- added R19: 191k, rcl:R0603
- added R20: 115k, rcl:R0603
- added R21: 3310Y-001-104L, 3310Y-001-104L:3310Y-001
- added R22: 1.58k, rcl:R0603
- added SWITCH_ALIM, SWITCH_SWD: MFS201N-9-Z, MFS201N-9-Z:MFS201N9Z
- added USB-ALIM: 10118193-0001LF, 10118193-0001LF:101181930001LF
- C20: value 0.1uF -> 100nF
- LED0, LED1, LED2, LED3, LED4, LED5, LED6, LED7: value (none) -> KPHD-1608LVQBC-D
- R10, R11, R12, R13, R6, R7, R8, R9: value (none) -> 330
- R14: value (none) -> 698
- moved SWD 17.1 mm to (96.5, 76.2), turned to 90 degrees
- moved R5 14.5 mm to (96.5, 64.8), turned to 0 degrees
- moved R4 11.5 mm to (96.5, 67.3), turned to 0 degrees
- moved R14 10.9 mm to (96.5, 62.2), turned to 0 degrees
- moved GPIO_TOP 9.25 mm to (73.7, 77.5)
- moved JPRF 7.62 mm to (16.5, 74.9)
- moved LED0 6.48 mm to (76.2, 68.6)
- moved LED2 6.48 mm to (71.1, 68.6)
- moved LED4 6.48 mm to (66.0, 68.6)
- moved R10 6.48 mm to (66.0, 64.8)
- moved R6 6.48 mm to (76.2, 64.8)
- moved R8 6.48 mm to (71.1, 64.8)
- moved LED3 6.48 mm to (68.6, 68.6)
- moved LED5 6.48 mm to (63.5, 68.6)
- moved LED6 6.48 mm to (61.0, 68.6)
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Connections:
- removed net VDDOUT: IC2.3
- removed net XIN: C18.1, IC2.142, Q1.1
- removed net XOUT: C19.1, IC2.141, Q1.2
- removed net _VDDCORE: IC3.5, JPCORE.1
- removed net _VDDMAIN: IC3.2, JPMAIN.1
- new net 2.2V: C23.1, FL1.5, R17.1, SWITCH_ALIM.3
- new net 5V: C26.1, C27.1, FL1.1, FL1.3, FL2.1, FL2.3, R22.2, USB-ALIM.1
- new net ALIM: SWITCH_ALIM.2, USBALIM.1
- new net N$14: C24.1, FL2.4, R19.2, R20.1
- new net N$15: C22.1, FL1.4, R17.2, R18.1
- new net N$16: R20.2, R21.2
- new net N$17: LED_2.2.A, SWITCH_ALIM.6
- new net N$18: R22.1, SWITCH_ALIM.5
- new net N$19: LED_VAR.A, SWITCH_ALIM.4
- new net VAR_V: C25.1, FL2.5, R19.1, SWITCH_ALIM.1
- net GND: now also C21.1, C22.2, C23.2, C24.2, C25.2, C26.2, C27.2, DBG_ON.C, FL1.2, FL2.2, JP1.2, LED_2.2.C, LED_VAR.C, R18.2, R21.1, SWITCH_SWD.1, USB-ALIM.5; no longer C1.2, C18.2, C19.2, C5.2, LED9.C
- net N$13: now also DBG_ON.A; no longer LED9.A
- net SWD_VCC: now also JP1.1, SWITCH_SWD.2; no longer IC3.3, IC3.6
- net VDDCORE: now also C21.2, IC2.3; no longer C5.1, JPCORE.2, JPVDD.2
- net VDDMAIN: now also SWITCH_SWD.3, USBALIM.2; no longer C1.1, JPMAIN.2, JPVDD.1
Routing:
- net ADD9: track 167.0 -> 49.6 mm, vias 6 -> 2
- net VDDCORE: track 171.2 -> 276.3 mm, vias 6 -> 9
- net NUB: track 55.0 -> 149.4 mm
- net DATA10: track 156.2 -> 63.7 mm, vias 0 -> 4
- net ADD16: track 38.8 -> 119.4 mm, vias 4 -> 6
- net 5V: track 0.00 -> 77.2 mm
- net SPI0_CS2: track 161.8 -> 91.9 mm, vias 3 -> 0
- net PHOTO: track 59.7 -> 117.5 mm, vias 4 -> 5
- net VDDMAIN: track 457.6 -> 401.8 mm, vias 11 -> 9
- net _VDDMAIN: track 54.6 -> 0.00 mm
- net _VDDCORE: track 52.6 -> 0.00 mm
- net ADD4: track 114.5 -> 71.5 mm, vias 6 -> 4
- net DATA12: track 31.5 -> 73.7 mm, vias 2 -> 6
- net GPIO_PA26: track 39.4 -> 80.7 mm, vias 3 -> 2
- net SPI0_CLK: track 125.8 -> 165.8 mm, vias 6 -> 4
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Other:
- board text added: "2.2V"
- board text added: "DBG ON"
- board text added: "SWD_VCC"
- board text added: "~V"
- board text removed: "+"
- board text removed: "IVCORE"
- board text removed: "IVDD"
- board text removed: "VCORE = VDD"
