File: eagle/base.sch (EAGLE design)
At the start: 70 parts, among them IC1 FM22L16-55-TG, IC2 ATSAMS70Q21A-AN, IC3 MFS401N-2-Z, IC4 ADT7310TRZ

Commit message: Update to version 2
Parts:
- removed C1, C5: 4.7uF, rcl:C-EUC0603
- removed C18, C19: (no value), rcl:C-EUC0603
- removed IC3: MFS401N-2-Z, MFS401N-2-Z:MFS401N-2-Z
- removed JPCORE, JPMAIN, JPVDD: (no value), pinhead:PINHD-1X2
- removed LED9: (no value), led:LEDCHIP-LED0603
- removed Q1: (no value), crystal:CRYSTALHC49S
- added C21: 100nF, rcl:C-EUC0603
- added C22, C24: 470pF, rcl:C-EUC0603
- added C23, C25: 2.2uF, rcl:C-EUC0603
- added C26, C27: 1uF, rcl:C-EUC0603
- added DBG_ON, LED_2.2, LED_VAR: KPHD-1608LVCGCK, led:LEDCHIP-LED0603
- added FL1, FL2: MIC5205YM5-TR, MIC5205YM5-TR:MIC5205YM5-TR
- added JP1, USBALIM: (no value), pinhead:PINHD-1X2
- added R17: 100k, rcl:R-US_R0603
- added R18: 76.8k, rcl:R-US_R0603
- added R19: 191k, rcl:R-US_R0603
- added R20: 115k, rcl:R-US_R0603
- added R21: 3310Y-001-104L, 3310Y-001-104L:3310Y-001-104L
- added R22: 1.58k, rcl:R-US_R0603
- added SWITCH_ALIM, SWITCH_SWD: MFS201N-9-Z, MFS201N-9-Z:MFS201N-9-Z
- added USB-ALIM: 10118193-0001LF, 10118193-0001LF:10118193-0001LF
- C20: value 0.1uF -> 100nF
- LED0, LED1, LED2, LED3, LED4, LED5, LED6, LED7: value (none) -> KPHD-1608LVQBC-D
- R10, R11, R12, R13, R6, R7, R8, R9: value (none) -> 330
- R14: value (none) -> 698
Connections:
- removed net XIN: C18.1, IC2.PB9, Q1.1
- removed net XOUT: C19.1, IC2.PB8, Q1.2
- removed net _VDDCORE: IC3.COM_2, JPCORE.1
- removed net _VDDMAIN: IC3.COM_1, JPMAIN.1
- new net 2.2V: C23.1, FL1.OUT, R17.1, SWITCH_ALIM.NC_1
- new net 5V: C26.1, C27.1, FL1.EN, FL1.IN, FL2.EN, FL2.IN, R22.2, USB-ALIM.1
- new net ALIM: SWITCH_ALIM.COM_1, USBALIM.1
- new net N$14: C24.1, FL2.ADJ, R19.2, R20.1
- new net N$15: C22.1, FL1.ADJ, R17.2, R18.1
- new net N$16: R20.2, R21.2
- new net N$17: LED_2.2.A, SWITCH_ALIM.NC_2
- new net N$18: R22.1, SWITCH_ALIM.COM_2
- new net N$19: LED_VAR.A, SWITCH_ALIM.NO_2
- new net VAR_V: C25.1, FL2.OUT, R19.1, SWITCH_ALIM.NO_1
- net GND: now also C21.1, C22.2, C23.2, C24.2, C25.2, C26.2, C27.2, DBG_ON.C, FL1.GND, FL2.GND, JP1.2, LED_2.2.C, LED_VAR.C, R18.2, R21.CCW, SWITCH_SWD.NO_1, USB-ALIM.5; no longer C1.2, C18.2, C19.2, C5.2, LED9.C
- net N$13: now also DBG_ON.A; no longer LED9.A
- net SWD_VCC: now also JP1.1, SWITCH_SWD.COM_1; no longer IC3.NO_1, IC3.NO_2
- net VDDCORE: now also C21.2, IC2.VDDOUT; no longer C5.1, JPCORE.2, JPVDD.2
- net VDDMAIN: now also SWITCH_SWD.NC_1, USBALIM.2; no longer C1.1, JPMAIN.2, JPVDD.1
Other:
- moved on the sheet: R14
